File: kicad/tapMatrix_Shield/tapMatrix.sch (KiCad schematic (older format))
At the start: 29 parts, among them IC1 DS1307, P5 TS_ZIF, P6 LED_MATRIX_HDR, P7 SPKR, U1 APE8865N-33-HF-3, U2 MCP4921-E/SN, U3 74LS125, U4 TL072, U5 SD_CARD

Commit message: begin routing pcb
Parts:
- U5: footprint (none) -> tapmatrix:114-00841-68
Changed lines of the file:
@@
 F 0 "U5" H 14750 2700 60  0000 C CNN
 F 1 "SD_CARD" H 14700 1300 60  0000 C CNN
-F 2 "" H 14700 2200 60  0001 C CNN
+F 2 "tapmatrix:114-00841-68" H 14700 2200 60  0001 C CNN
 F 3 "" H 14700 2200 60  0000 C CNN
 	1    14700 2000
@@
 Wire Wire Line
 	11750 2750 11750 3050
+Connection ~ 10600 4650
 $EndSCHEMATC

Commit message: continue routing
Connections:
- net labels added: DATA_IN
Changed lines of the file:
@@
 MISO
 Text Label 10650 2600 0    60   ~ 0
-MISO
+DATA_IN
 Text Label 9400 2600 0    60   ~ 0
 MOSI
@@
 CS
 Text Label 13650 1900 0    60   ~ 0
-MOSI
+DATA_IN
 Text Label 3550 1550 0    60   ~ 0
 SD_CS

Commit message: removed volume pot; created gerber files
Parts:
- removed RV1: POT, symbol POT
Other:
- note added: "(VOLUME REMOVED)"
- note removed: "VOLUME"
Changed lines of the file:
@@
-$EndComp
-$Comp
-L POT RV1
-U 1 1 53F6D006
-P 11100 4900
-F 0 "RV1" H 11100 4800 50  0000 C CNN
-F 1 "POT" H 11100 4900 50  0000 C CNN
-F 2 "" H 11100 4900 60  0001 C CNN
-F 3 "" H 11100 4900 60  0000 C CNN
-	1    11100 4900
-	0    1    1    0
 $EndComp
 $Comp
@@
 $EndComp
 $Comp
-L GND #PWR016
-U 1 1 53F6D161
-P 11100 5450
-F 0 "#PWR016" H 11100 5450 30  0001 C CNN
-F 1 "GND" H 11100 5380 30  0001 C CNN
-F 2 "" H 11100 5450 60  0000 C CNN
-F 3 "" H 11100 5450 60  0000 C CNN
-	1    11100 5450
-	1    0    0    -1
-$EndComp
-$Comp
 L TL072 U4
 U 1 1 53F6DDA6
@@
 $EndComp
 $Comp
-L GND #PWR017
+L GND #PWR016
 U 1 1 53F6E130
 P 14000 5550
-F 0 "#PWR017" H 14000 5550 30  0001 C CNN
+F 0 "#PWR016" H 14000 5550 30  0001 C CNN
 F 1 "GND" H 14000 5480 30  0001 C CNN
 F 2 "" H 14000 5550 60  0000 C CNN
@@
 $EndComp
 $Comp
-L GND #PWR018
+L GND #PWR017
 U 1 1 53F6E684
 P 15900 5750
-F 0 "#PWR018" H 15900 5750 30  0001 C CNN
+F 0 "#PWR017" H 15900 5750 30  0001 C CNN
 F 1 "GND" H 15900 5680 30  0001 C CNN
 F 2 "" H 15900 5750 60  0000 C CNN
@@
 $EndComp
 $Comp
-L +5V #PWR019
+L +5V #PWR018
 U 1 1 53F6EE99
 P 3550 4800
-F 0 "#PWR019" H 3550 4890 20  0001 C CNN
+F 0 "#PWR018" H 3550 4890 20  0001 C CNN
 F 1 "+5V" H 3550 4890 30  0000 C CNN
 F 2 "" H 3550 4800 60  0000 C CNN
@@
 $EndComp
 $Comp
-L GND #PWR020
+L GND #PWR019
 U 1 1 53F6F180
 P 4200 5400
-F 0 "#PWR020" H 4200 5400 30  0001 C CNN
+F 0 "#PWR019" H 4200 5400 30  0001 C CNN
 F 1 "GND" H 4200 5330 30  0001 C CNN
 F 2 "" H 4200 5400 60  0000 C CNN
@@
 $EndComp
 $Comp
-L +3.3V #PWR021
+L +3.3V #PWR020
 U 1 1 53F6F2EF
 P 5050 4800
-F 0 "#PWR021" H 5050 4760 30  0001 C CNN
+F 0 "#PWR020" H 5050 4760 30  0001 C CNN
 F 1 "+3.3V" H 5050 4910 30  0000 C CNN
 F 2 "" H 5050 4800 60  0000 C CNN
@@
 $EndComp
 $Comp
-L GND #PWR022
+L GND #PWR021
 U 1 1 53F6F8C4
 P 3100 5300
-F 0 "#PWR022" H 3100 5300 30  0001 C CNN
+F 0 "#PWR021" H 3100 5300 30  0001 C CNN
 F 1 "GND" H 3100 5230 30  0001 C CNN
 F 2 "" H 3100 5300 60  0000 C CNN
@@
 NoConn ~ 1650 1150
 $Comp
-L GND #PWR023
+L GND #PWR022
 U 1 1 53F7124A
 P 2200 5300
-F 0 "#PWR023" H 2200 5300 30  0001 C CNN
+F 0 "#PWR022" H 2200 5300 30  0001 C CNN
 F 1 "GND" H 2200 5230 30  0001 C CNN
 F 2 "" H 2200 5300 60  0000 C CNN
@@
 $EndComp
 $Comp
-L GND #PWR024
+L GND #PWR023
 U 1 1 53F7125E
 P 2500 5300
-F 0 "#PWR024" H 2500 5300 30  0001 C CNN
+F 0 "#PWR023" H 2500 5300 30  0001 C CNN
 F 1 "GND" H 2500 5230 30  0001 C CNN
 F 2 "" H 2500 5300 60  0000 C CNN
@@
 Text Notes 12900 5800 0    60   ~ 0
 AMP
-Text Notes 11000 5800 0    60   ~ 0
-VOLUME
+Text Notes 11050 5800 0    60   ~ 0
+(VOLUME REMOVED)
 $Comp
 L DS1307 IC1
@@
 	10600 4650 11100 4650
 Wire Wire Line
-	11100 5150 11100 5450
-Wire Wire Line
 	13600 5100 13600 5650
 Wire Wire Line
@@
 Connection ~ 13100 5500
 Wire Wire Line
-	11250 4900 12100 4900
+	11100 4900 12100 4900
 Connection ~ 12100 4900
 Wire Wire Line
@@
 $EndComp
 $Comp
-L GND #PWR025
+L GND #PWR024
 U 1 1 53F7C63E
 P 2450 8000
-F 0 "#PWR025" H 2450 8000 30  0001 C CNN
+F 0 "#PWR024" H 2450 8000 30  0001 C CNN
 F 1 "GND" H 2450 7930 30  0001 C CNN
 F 2 "" H 2450 8000 60  0000 C CNN
@@
 NoConn ~ 1650 1050
 $Comp
-L +5V #PWR026
+L +5V #PWR025
 U 1 1 53F94A7D
 P 2200 4550
-F 0 "#PWR026" H 2200 4640 20  0001 C CNN
+F 0 "#PWR025" H 2200 4640 20  0001 C CNN
 F 1 "+5V" H 2200 4640 30  0000 C CNN
 F 2 "" H 2200 4550 60  0000 C CNN
@@
 	2200 4550 2200 4800
 $Comp
-L +5V #PWR027
+L +5V #PWR026
 U 1 1 53F94B8C
 P 2500 4550
-F 0 "#PWR027" H 2500 4640 20  0001 C CNN
+F 0 "#PWR026" H 2500 4640 20  0001 C CNN
 F 1 "+5V" H 2500 4640 30  0000 C CNN
 F 2 "" H 2500 4550 60  0000 C CNN
@@
 	2500 4550 2500 4800
 $Comp
-L +5V #PWR028
+L +5V #PWR027
 U 1 1 53F94C7A
 P 3100 4550
-F 0 "#PWR028" H 3100 4640 20  0001 C CNN
+F 0 "#PWR027" H 3100 4640 20  0001 C CNN
 F 1 "+5V" H 3100 4640 30  0000 C CNN
 F 2 "" H 3100 4550 60  0000 C CNN
@@
 NoConn ~ 3450 1750
 $Comp
-L +5V #PWR029
+L +5V #PWR028
 U 1 1 53F96D63
 P 9300 4000
-F 0 "#PWR029" H 9300 4090 20  0001 C CNN
+F 0 "#PWR028" H 9300 4090 20  0001 C CNN
 F 1 "+5V" H 9300 4090 30  0000 C CNN
 F 2 "" H 9300 4000 60  0000 C CNN
@@
 NoConn ~ 3450 1050
 $Comp
-L GND #PWR030
+L GND #PWR029
 U 1 1 53F9875B
 P 4050 1250
-F 0 "#PWR030" H 4050 1250 30  0001 C CNN
+F 0 "#PWR029" H 4050 1250 30  0001 C CNN
 F 1 "GND" H 4050 1180 30  0001 C CNN
 F 2 "" H 4050 1250 60  0000 C CNN
@@
 	9950 1300 9950 1500
 $Comp
-L GND #PWR031
+L GND #PWR030
 U 1 1 53F9AF0C
 P 10100 2100
-F 0 "#PWR031" H 10100 2100 30  0001 C CNN
+F 0 "#PWR030" H 10100 2100 30  0001 C CNN
 F 1 "GND" H 10100 2030 30  0001 C CNN
 F 2 "" H 10100 2100 60  0000 C CNN
@@
 $EndComp
 $Comp
-L GND #PWR032
+L GND #PWR031
 U 1 1 53F9B0AC
 P 10100 3050
-F 0 "#PWR032" H 10100 3050 30  0001 C CNN
+F 0 "#PWR031" H 10100 3050 30  0001 C CNN
 F 1 "GND" H 10100 2980 30  0001 C CNN
 F 2 "" H 10100 3050 60  0000 C CNN
@@
 $EndComp
 $Comp
-L GND #PWR033
+L GND #PWR032
 U 1 1 53F9B165
 P 11900 2100
-F 0 "#PWR033" H 11900 2100 30  0001 C CNN
+F 0 "#PWR032" H 11900 2100 30  0001 C CNN
 F 1 "GND" H 11900 2030 30  0001 C CNN
 F 2 "" H 11900 2100 60  0000 C CNN
@@
 	11450 1450 11450 1650
 $Comp
-L +5V #PWR034
+L +5V #PWR033
 U 1 1 53F9B69B
 P 11450 800
-F 0 "#PWR034" H 11450 890 20  0001 C CNN
+F 0 "#PWR033" H 11450 890 20  0001 C CNN
 F 1 "+5V" H 11450 890 30  0000 C CNN
 F 2 "" H 11450 800 60  0000 C CNN
@@
 	9950 2300 9950 2450
 $Comp
-L +3.3V #PWR035
+L +3.3V #PWR034
 U 1 1 53F9C9E7
 P 11750 2250
-F 0 "#PWR035" H 11750 2210 30  0001 C CNN
+F 0 "#PWR034" H 11750 2210 30  0001 C CNN
 F 1 "+3.3V" H 11750 2360 30  0000 C CNN
 F 2 "" H 11750 2250 60  0000 C CNN
@@
 	11750 2250 11750 2450
 $Comp
-L GND #PWR036
+L GND #PWR035
 U 1 1 53F9CBA6
 P 11750 3050
-F 0 "#PWR036" H 11750 3050 30  0001 C CNN
+F 0 "#PWR035" H 11750 3050 30  0001 C CNN
 F 1 "GND" H 11750 2980 30  0001 C CNN
 F 2 "" H 11750 3050 60  0000 C CNN
@@
 	1150 1250 1650 1250
 $Comp
-L +5V #PWR037
+L +5V #PWR036
 U 1 1 53F9E6C1
 P 14000 4350
-F 0 "#PWR037" H 14000 4440 20  0001 C CNN
+F 0 "#PWR036" H 14000 4440 20  0001 C CNN
 F 1 "+5V" H 14000 4440 30  0000 C CNN
 F 2 "" H 14000 4350 60  0000 C CNN
@@
 	11750 2750 11750 3050
 Connection ~ 10600 4650
+Wire Wire Line
+	11100 4650 11100 4900
 $EndSCHEMATC

Commit message: added optional 4-pin header as alt for touchscreen zif
Parts:
- added JP5: 4_PIN_1, Pin_Headers:Pin_Header_Straight_1x04, symbol 4_PIN_1
- C4, C6, C9: footprint Capacitors_SMD:c_0603 -> Capacitors_Tantalum_SMD:TantalC_SizeC_EIA-6032_Reflow
- renumbered P7 to JP6
Connections:
- wire segments 133 -> 137
Other:
- note added: "Touchscreen ZIF Socket + Optional Header"
- note removed: "Touchscreen ZIF Socket"
Changed lines of the file:
@@
 L TS_ZIF P5
 U 1 1 53F23B9F
-P 5300 2550
-F 0 "P5" H 5350 2850 50  0000 C CNN
-F 1 "TS_ZIF" V 5500 2550 50  0000 C CNN
-F 2 "tapmatrix:SFW4R­5STE1LF" H 5300 2550 60  0001 C CNN
-F 3 "" H 5300 2550 60  0000 C CNN
-	1    5300 2550
+P 5000 2550
+F 0 "P5" H 5050 2850 50  0000 C CNN
+F 1 "TS_ZIF" V 5200 2550 50  0000 C CNN
+F 2 "tapmatrix:SFW4R­5STE1LF" H 5000 2550 60  0001 C CNN
+F 3 "" H 5000 2550 60  0000 C CNN
+	1    5000 2550
 	1    0    0    -1
 $EndComp
@@
 	1    0    0    -1
 $EndComp
-Text Notes 5500 3250 2    60   ~ 0
-Touchscreen ZIF Socket
+Text Notes 6500 3250 2    60   ~ 0
+Touchscreen ZIF Socket + Optional Header
 Text Notes 8000 3250 2    60   ~ 0
 LED Matrix Header
@@
 Text Label 1350 2500 0    60   ~ 0
 YM
-Text Label 4700 2400 0    60   ~ 0
+Text Label 4400 2400 0    60   ~ 0
 XM
-Text Label 4700 2500 0    60   ~ 0
+Text Label 4400 2500 0    60   ~ 0
 YP
-Text Label 4700 2600 0    60   ~ 0
+Text Label 4400 2600 0    60   ~ 0
 XP
-Text Label 4700 2700 0    60   ~ 0
+Text Label 4400 2700 0    60   ~ 0
 YM
 Text Label 15400 1900 0    60   ~ 0
@@
 F 0 "C9" H 15100 5100 40  0000 L CNN
 F 1 "100uF/6V" H 15106 4915 40  0000 L CNN
-F 2 "Capacitors_SMD:c_0603" H 15138 4850 30  0001 C CNN
+F 2 "Capacitors_Tantalum_SMD:TantalC_SizeC_EIA-6032_Reflow" H 15138 4850 30  0001 C CNN
 F 3 "" H 15100 5000 60  0000 C CNN
 	1    15100 5000
@@
 $EndComp
 $Comp
-L CONN_2 P7
+L CONN_2 JP6
 U 1 1 53F6E48F
 P 15550 5500
-F 0 "P7" V 15500 5500 40  0000 C CNN
+F 0 "JP6" V 15500 5500 40  0000 C CNN
 F 1 "SPKR" V 15600 5500 40  0000 C CNN
 F 2 "Pin_Headers:Pin_Header_Straight_1x02" H 15550 5500 60  0001 C CNN
@@
 F 0 "C6" H 5400 5100 40  0000 L CNN
 F 1 "100uF/6V" H 5406 4915 40  0000 L CNN
-F 2 "Capacitors_SMD:c_0603" H 5438 4850 30  0001 C CNN
+F 2 "Capacitors_Tantalum_SMD:TantalC_SizeC_EIA-6032_Reflow" H 5438 4850 30  0001 C CNN
 F 3 "" H 5400 5000 60  0000 C CNN
 	1    5400 5000
@@
 F 0 "C4" H 3100 5100 40  0000 L CNN
 F 1 "100uF/6V" H 3106 4915 40  0000 L CNN
-F 2 "Capacitors_SMD:c_0603" H 3138 4850 30  0001 C CNN
+F 2 "Capacitors_Tantalum_SMD:TantalC_SizeC_EIA-6032_Reflow" H 3138 4850 30  0001 C CNN
 F 3 "" H 3100 5000 60  0000 C CNN
 	1    3100 5000
@@
 $EndComp
 Wire Wire Line
-	4700 2700 4950 2700
-Wire Wire Line
-	4700 2500 4950 2500
+	4400 2700 4650 2700
+Wire Wire Line
+	4400 2500 4650 2500
 Wire Wire Line
 	-766900 -630300 -767100 -630300
@@
 	1650 2400 1350 2400
 Wire Wire Line
-	4950 2400 4700 2400
-Wire Wire Line
-	4950 2600 4700 2600
+	4650 2400 4400 2400
+Wire Wire Line
+	4650 2600 4400 2600
 Wire Wire Line
 	14000 1900 13650 1900
@@
 Wire Wire Line
 	11100 4650 11100 4900
+$Comp
+L 4_PIN_1 JP5
+U 1 1 5407DC2F
+P 6250 2550
+F 0 "JP5" H 6250 2850 60  0000 C CNN
+F 1 "4_PIN_1" V 6350 2550 60  0000 C CNN
+F 2 "Pin_Headers:Pin_Header_Straight_1x04" H 6250 2550 60  0001 C CNN
+F 3 "" H 6250 2550 60  0000 C CNN
+	1    6250 2550
+	1    0    0    -1
+$EndComp
+Wire Wire Line
+	5800 2400 5500 2400
+Wire Wire Line
+	5800 2500 5500 2500
+Wire Wire Line
+	5800 2600 5500 2600
+Wire Wire Line
+	5800 2700 5500 2700
+Text Label 5500 2400 0    60   ~ 0
+XM
+Text Label 5500 2500 0    60   ~ 0
+YP
+Text Label 5500 2600 0    60   ~ 0
+XP
+Text Label 5500 2700 0    60   ~ 0
+YM
 $EndSCHEMATC

Commit message: replace voltage regulator with corrected component
Parts:
- U1: value APE8865N-33-HF-3 -> MCP1700T-3302E/MB; footprint SMD_Packages:SOT-23 -> Housings_SOT-89:SOT89-3_Housing
Changed lines of the file:
@@
 Sheet 1 1
 Title "tapMatrix Shield"
-Date "17 Aug 2014"
-Rev "0.1"
+Date "03 Sep 2014"
+Rev "0.2"
 Comp "Responsive Devices, Inc."
 Comment1 ""
@@
 P 4200 4850
 F 0 "U1" H 3900 5100 40  0000 C CNN
-F 1 "APE8865N-33-HF-3" H 4200 5050 40  0000 C CNN
-F 2 "SMD_Packages:SOT-23" H 4200 4950 35  0000 C CIN
+F 1 "MCP1700T-3302E/MB" H 4200 5050 40  0000 C CNN
+F 2 "Housings_SOT-89:SOT89-3_Housing" H 4200 5200 35  0001 C CIN
 F 3 "" H 4200 4850 60  0000 C CNN
 	1    4200 4850

Commit message: create v0.3_ fix problems with U1, U3, U4 components U1 used the wrong footprint. changed from SOT-23 to SOT-89-3 U3 used the narrow version of SOIC-14 (incorrectly named in library as SOIC-14_W). changed to actual SOIC-14-Wide U4 incorrectly used SOIC-14 footprint. changed to SOIC-8 tore up the layout, placed new footprints. still need to reroute everything
Parts:
- U3: footprint SMD_Packages:SOIC-14_W -> SMD_Packages:SOIC-14_N
- U4: footprint SMD_Packages:SOIC-14_N -> Housings_SOIC:SOIC-8_N
Changed lines of the file:
@@
 Sheet 1 1
 Title "tapMatrix Shield"
-Date "03 Sep 2014"
-Rev "0.2"
+Date "22 Sep 2014"
+Rev "0.3"
 Comp "Responsive Devices, Inc."
 Comment1 ""
@@
 F 0 "U3" H 10100 1750 50  0000 L BNN
 F 1 "74LS125" H 10150 1500 40  0000 L TNN
-F 2 "SMD_Packages:SOIC-14_W" H 10100 1650 60  0001 C CNN
+F 2 "SMD_Packages:SOIC-14_N" H 10100 1650 60  0001 C CNN
 F 3 "" H 10100 1650 60  0000 C CNN
 	1    10100 1650
@@
 F 0 "U3" H 11900 1750 50  0000 L BNN
 F 1 "74LS125" H 11950 1500 40  0000 L TNN
-F 2 "SMD_Packages:SOIC-14_W" H 11900 1650 60  0001 C CNN
+F 2 "SMD_Packages:SOIC-14_N" H 11900 1650 60  0001 C CNN
 F 3 "" H 11900 1650 60  0000 C CNN
 	3    11900 1650
@@
 F 0 "U3" H 10100 2700 50  0000 L BNN
 F 1 "74LS125" H 10150 2450 40  0000 L TNN
-F 2 "SMD_Packages:SOIC-14_W" H 10100 2600 60  0001 C CNN
+F 2 "SMD_Packages:SOIC-14_N" H 10100 2600 60  0001 C CNN
 F 3 "" H 10100 2600 60  0000 C CNN
 	2    10100 2600
@@
 F 0 "U3" H 11900 2700 50  0000 L BNN
 F 1 "74LS125" H 11950 2450 40  0000 L TNN
-F 2 "SMD_Packages:SOIC-14_W" H 11900 2600 60  0001 C CNN
+F 2 "SMD_Packages:SOIC-14_N" H 11900 2600 60  0001 C CNN
 F 3 "" H 11900 2600 60  0000 C CNN
 	4    11900 2600
@@
 U 1 1 53F6C019
 P 9400 4650
-F 0 "U2" H 9400 5000 40  0000 L BNN
-F 1 "MCP4921-E/SN" H 9400 4950 40  0000 L BNN
-F 2 "SMD_Packages:SOIC-8-N" H 9400 4650 30  0000 C CIN
+F 0 "U2" H 9400 5050 40  0000 L BNN
+F 1 "MCP4921-E/SN" H 9400 5000 40  0000 L BNN
+F 2 "SMD_Packages:SOIC-8-N" H 9700 4950 30  0000 C CIN
 F 3 "" H 9400 4650 60  0000 C CNN
 	1    9400 4650
@@
 F 0 "U4" H 12550 5200 60  0000 L CNN
 F 1 "TL072" H 12550 4750 60  0000 L CNN
-F 2 "SMD_Packages:SOIC-14_N" H 12600 5000 60  0001 C CNN
+F 2 "Housings_SOIC:SOIC-8_N" H 12600 5000 60  0001 C CNN
 F 3 "" H 12600 5000 60  0000 C CNN
 	1    12600 5000
@@
 F 0 "U4" H 14050 5200 60  0000 L CNN
 F 1 "TL072" H 14050 4750 60  0000 L CNN
-F 2 "SMD_Packages:SOIC-14_N" H 14100 5000 60  0001 C CNN
+F 2 "Housings_SOIC:SOIC-8_N" H 14100 5000 60  0001 C CNN
 F 3 "" H 14100 5000 60  0000 C CNN
 	2    14100 5000

Commit message: Revised r0.3 components, tore up pcb
Parts:
- C4, C6, C9: footprint Capacitors_Tantalum_SMD:TantalC_SizeC_EIA-6032_Reflow -> tapmatrix:EEE-0JA101WR
- U6: renamed from IC1; footprint Housings_SOIC:SOIC-8_N -> tapmatrix:SOIC-8_N
Changed lines of the file:
@@
 Sheet 1 1
 Title "tapMatrix Shield"
-Date "22 Sep 2014"
+Date "26 Oct 2014"
 Rev "0.3"
 Comp "Responsive Devices, Inc."
@@
 F 0 "C9" H 15100 5100 40  0000 L CNN
 F 1 "100uF/6V" H 15106 4915 40  0000 L CNN
-F 2 "Capacitors_Tantalum_SMD:TantalC_SizeC_EIA-6032_Reflow" H 15138 4850 30  0001 C CNN
+F 2 "tapmatrix:EEE-0JA101WR" H 15138 4850 30  0001 C CNN
 F 3 "" H 15100 5000 60  0000 C CNN
 	1    15100 5000
@@
 F 0 "C6" H 5400 5100 40  0000 L CNN
 F 1 "100uF/6V" H 5406 4915 40  0000 L CNN
-F 2 "Capacitors_Tantalum_SMD:TantalC_SizeC_EIA-6032_Reflow" H 5438 4850 30  0001 C CNN
+F 2 "tapmatrix:EEE-0JA101WR" H 5438 4850 30  0001 C CNN
 F 3 "" H 5400 5000 60  0000 C CNN
 	1    5400 5000
@@
 F 0 "C4" H 3100 5100 40  0000 L CNN
 F 1 "100uF/6V" H 3106 4915 40  0000 L CNN
-F 2 "Capacitors_Tantalum_SMD:TantalC_SizeC_EIA-6032_Reflow" H 3138 4850 30  0001 C CNN
+F 2 "tapmatrix:EEE-0JA101WR" H 3138 4850 30  0001 C CNN
 F 3 "" H 3100 5000 60  0000 C CNN
 	1    3100 5000
@@
 (VOLUME REMOVED)
 $Comp
-L DS1307 IC1
+L DS1307 U6
 U 1 1 53F71D16
 P 3650 7650
-F 0 "IC1" H 3650 7450 60  0000 C CNN
+F 0 "U6" H 3650 7450 60  0000 C CNN
 F 1 "DS1307" H 3650 7900 60  0000 C CNN
-F 2 "Housings_SOIC:SOIC-8_N" H 3650 7650 60  0001 C CNN
+F 2 "tapmatrix:SOIC-8_N" H 3650 7650 60  0001 C CNN
 F 3 "" H 3650 7650 60  0000 C CNN
 	1    3650 7650
@@
 Wire Wire Line
 	5500 6700 5500 6900
-Wire Wire Line
-	4450 7700 5850 7700
 Wire Wire Line
 	5500 7700 5500 7400
@@
 Text Label 5500 2700 0    60   ~ 0
 YM
+Wire Wire Line
+	4450 7700 5850 7700
 $EndSCHEMATC

Commit message: corrected error with U1 pins (2 and 3 were reversed)
Parts:
- C1, C2, C3, C5, C7, C8: footprint Capacitors_SMD:c_0603 -> tapmatrix:C_0603
- JP1, JP2: footprint Pin_Headers:Pin_Header_Straight_1x06 -> tapmatrix:Pin_Header_Straight_1x06
- JP3, JP4: footprint Pin_Headers:Pin_Header_Straight_1x08 -> tapmatrix:Pin_Header_Straight_1x08
- JP5: footprint Pin_Headers:Pin_Header_Straight_1x04 -> tapmatrix:Pin_Header_Straight_1x04
- JP6: footprint Pin_Headers:Pin_Header_Straight_1x02 -> tapmatrix:Pin_Header_Straight_1x02
- R1, R2, R3, R4, R5: footprint Resistors_SMD:R_0603 -> tapmatrix:R_0603
- U1: footprint Housings_SOT-89:SOT89-3_Housing -> tapmatrix:SOT89-3_Housing
- U2: footprint SMD_Packages:SOIC-8-N -> tapmatrix:SOIC-8_N
- U3: footprint SMD_Packages:SOIC-14_N -> tapmatrix:SO-14
- U4: footprint Housings_SOIC:SOIC-8_N -> tapmatrix:SOIC-8_N
Changed lines of the file:
@@
 F 0 "U3" H 10100 1750 50  0000 L BNN
 F 1 "74LS125" H 10150 1500 40  0000 L TNN
-F 2 "SMD_Packages:SOIC-14_N" H 10100 1650 60  0001 C CNN
+F 2 "tapmatrix:SO-14" H 10100 1650 60  0001 C CNN
 F 3 "" H 10100 1650 60  0000 C CNN
 	1    10100 1650
@@
 F 0 "U3" H 11900 1750 50  0000 L BNN
 F 1 "74LS125" H 11950 1500 40  0000 L TNN
-F 2 "SMD_Packages:SOIC-14_N" H 11900 1650 60  0001 C CNN
+F 2 "tapmatrix:SO-14" H 11900 1650 60  0001 C CNN
 F 3 "" H 11900 1650 60  0000 C CNN
 	3    11900 1650
@@
 F 0 "U3" H 10100 2700 50  0000 L BNN
 F 1 "74LS125" H 10150 2450 40  0000 L TNN
-F 2 "SMD_Packages:SOIC-14_N" H 10100 2600 60  0001 C CNN
+F 2 "tapmatrix:SO-14" H 10100 2600 60  0001 C CNN
 F 3 "" H 10100 2600 60  0000 C CNN
 	2    10100 2600
@@
 F 0 "U3" H 11900 2700 50  0000 L BNN
 F 1 "74LS125" H 11950 2450 40  0000 L TNN
-F 2 "SMD_Packages:SOIC-14_N" H 11900 2600 60  0001 C CNN
+F 2 "tapmatrix:SO-14" H 11900 2600 60  0001 C CNN
 F 3 "" H 11900 2600 60  0000 C CNN
 	4    11900 2600
@@
 F 0 "R5" V 11530 1200 40  0000 C CNN
 F 1 "10K" V 11457 1201 40  0000 C CNN
-F 2 "Resistors_SMD:R_0603" V 11380 1200 30  0001 C CNN
+F 2 "tapmatrix:R_0603" V 11380 1200 30  0001 C CNN
 F 3 "" H 11450 1200 30  0000 C CNN
 	1    11450 1200
@@
 F 0 "JP1" H 2100 1650 60  0000 C CNN
 F 1 "6_PIN_1" H 2100 950 60  0000 C CNN
-F 2 "Pin_Headers:Pin_Header_Straight_1x06" H 2000 1300 60  0001 C CNN
+F 2 "tapmatrix:Pin_Header_Straight_1x06" H 2000 1300 60  0001 C CNN
 F 3 "" H 2000 1300 60  0000 C CNN
 	1    2000 1300
@@
 F 0 "JP2" H 2100 2800 60  0000 C CNN
 F 1 "6_PIN_2" H 2100 2100 60  0000 C CNN
-F 2 "Pin_Headers:Pin_Header_Straight_1x06" H 2000 2450 60  0001 C CNN
+F 2 "tapmatrix:Pin_Header_Straight_1x06" H 2000 2450 60  0001 C CNN
 F 3 "" H 2000 2450 60  0000 C CNN
 	1    2000 2450
@@
 F 0 "JP3" H 3000 1850 60  0000 C CNN
 F 1 "8_PIN_1" H 3000 950 60  0000 C CNN
-F 2 "Pin_Headers:Pin_Header_Straight_1x08" H 2900 1500 60  0001 C CNN
+F 2 "tapmatrix:Pin_Header_Straight_1x08" H 2900 1500 60  0001 C CNN
 F 3 "" H 2900 1500 60  0000 C CNN
 	1    2900 1400
@@
 F 0 "JP4" H 3000 3000 60  0000 C CNN
 F 1 "8_PIN_2" H 3000 2100 60  0000 C CNN
-F 2 "Pin_Headers:Pin_Header_Straight_1x08" H 2900 2650 60  0001 C CNN
+F 2 "tapmatrix:Pin_Header_Straight_1x08" H 2900 2650 60  0001 C CNN
 F 3 "" H 2900 2650 60  0000 C CNN
 	1    2900 2550
@@
 F 0 "U2" H 9400 5050 40  0000 L BNN
 F 1 "MCP4921-E/SN" H 9400 5000 40  0000 L BNN
-F 2 "SMD_Packages:SOIC-8-N" H 9700 4950 30  0000 C CIN
+F 2 "tapmatrix:SOIC-8_N" H 9700 4950 30  0000 C CIN
 F 3 "" H 9400 4650 60  0000 C CNN
 	1    9400 4650
@@
 F 0 "C7" H 9750 5350 40  0000 L CNN
 F 1 "0.1uF" H 9756 5165 40  0000 L CNN
-F 2 "Capacitors_SMD:c_0603" H 9788 5100 30  0001 C CNN
+F 2 "tapmatrix:C_0603" H 9788 5100 30  0001 C CNN
 F 3 "" H 9750 5250 60  0000 C CNN
 	1    9750 5250
@@
 F 0 "R3" V 10080 5050 40  0000 C CNN
 F 1 "100K" V 10007 5051 40  0000 C CNN
-F 2 "Resistors_SMD:R_0603" V 9930 5050 30  0001 C CNN
+F 2 "tapmatrix:R_0603" V 9930 5050 30  0001 C CNN
 F 3 "" H 10000 5050 30  0000 C CNN
 	1    10000 5050
@@
 F 0 "R4" V 10430 4650 40  0000 C CNN
 F 1 "1.5K" V 10357 4651 40  0000 C CNN
-F 2 "Resistors_SMD:R_0603" V 10280 4650 30  0001 C CNN
+F 2 "tapmatrix:R_0603" V 10280 4650 30  0001 C CNN
 F 3 "" H 10350 4650 30  0000 C CNN
 	1    10350 4650
@@
 F 0 "C8" H 10600 5350 40  0000 L CNN
 F 1 "0.01uF" H 10606 5165 40  0000 L CNN
-F 2 "Capacitors_SMD:c_0603" H 10638 5100 30  0001 C CNN
+F 2 "tapmatrix:C_0603" H 10638 5100 30  0001 C CNN
 F 3 "" H 10600 5250 60  0000 C CNN
 	1    10600 5250
@@
 F 0 "U4" H 12550 5200 60  0000 L CNN
 F 1 "TL072" H 12550 4750 60  0000 L CNN
-F 2 "Housings_SOIC:SOIC-8_N" H 12600 5000 60  0001 C CNN
+F 2 "tapmatrix:SOIC-8_N" H 12600 5000 60  0001 C CNN
 F 3 "" H 12600 5000 60  0000 C CNN
 	1    12600 5000
@@
 F 0 "U4" H 14050 5200 60  0000 L CNN
 F 1 "TL072" H 14050 4750 60  0000 L CNN
-F 2 "Housings_SOIC:SOIC-8_N" H 14100 5000 60  0001 C CNN
+F 2 "tapmatrix:SOIC-8_N" H 14100 5000 60  0001 C CNN
 F 3 "" H 14100 5000 60  0000 C CNN
 	2    14100 5000
@@
 F 0 "JP6" V 15500 5500 40  0000 C CNN
 F 1 "SPKR" V 15600 5500 40  0000 C CNN
-F 2 "Pin_Headers:Pin_Header_Straight_1x02" H 15550 5500 60  0001 C CNN
+F 2 "tapmatrix:Pin_Header_Straight_1x02" H 15550 5500 60  0001 C CNN
 F 3 "" H 15550 5500 60  0000 C CNN
 	1    15550 5500
@@
 F 0 "U1" H 3900 5100 40  0000 C CNN
 F 1 "MCP1700T-3302E/MB" H 4200 5050 40  0000 C CNN
-F 2 "Housings_SOT-89:SOT89-3_Housing" H 4200 5200 35  0001 C CIN
+F 2 "tapmatrix:SOT89-3_Housing" H 4200 5200 35  0001 C CIN
 F 3 "" H 4200 4850 60  0000 C CNN
 	1    4200 4850
@@
 F 0 "C5" H 4650 5100 40  0000 L CNN
 F 1 "0.1uF" H 4656 4915 40  0000 L CNN
-F 2 "Capacitors_SMD:c_0603" H 4688 4850 30  0001 C CNN
+F 2 "tapmatrix:C_0603" H 4688 4850 30  0001 C CNN
 F 3 "" H 4650 5000 60  0000 C CNN
 	1    4650 5000
@@
 F 0 "C2" H 2500 5100 40  0000 L CNN
 F 1 "0.1uF" H 2506 4915 40  0000 L CNN
-F 2 "Capacitors_SMD:c_0603" H 2538 4850 30  0001 C CNN
+F 2 "tapmatrix:C_0603" H 2538 4850 30  0001 C CNN
 F 3 "" H 2500 5000 60  0000 C CNN
 	1    2500 5000
@@
 F 0 "C3" H 2800 5100 40  0000 L CNN
 F 1 "0.1uF" H 2806 4915 40  0000 L CNN
-F 2 "Capacitors_SMD:c_0603" H 2838 4850 30  0001 C CNN
+F 2 "tapmatrix:C_0603" H 2838 4850 30  0001 C CNN
 F 3 "" H 2800 5000 60  0000 C CNN
 	1    2800 5000
@@
 F 0 "C1" H 2200 5100 40  0000 L CNN
 F 1 "0.1uF" H 2206 4915 40  0000 L CNN
-F 2 "Capacitors_SMD:c_0603" H 2238 4850 30  0001 C CNN
+F 2 "tapmatrix:C_0603" H 2238 4850 30  0001 C CNN
 F 3 "" H 2200 5000 60  0000 C CNN
 	1    2200 5000
@@
 F 0 "R1" V 4930 7150 40  0000 C CNN
 F 1 "R" V 4857 7151 40  0000 C CNN
-F 2 "Resistors_SMD:R_0603" V 4780 7150 30  0001 C CNN
+F 2 "tapmatrix:R_0603" V 4780 7150 30  0001 C CNN
 F 3 "" H 4850 7150 30  0000 C CNN
 	1    4850 7150
@@
 F 0 "R2" V 5580 7150 40  0000 C CNN
 F 1 "R" V 5507 7151 40  0000 C CNN
-F 2 "Resistors_SMD:R_0603" V 5430 7150 30  0001 C CNN
+F 2 "tapmatrix:R_0603" V 5430 7150 30  0001 C CNN
 F 3 "" H 5500 7150 30  0000 C CNN
 	1    5500 7150
@@
 F 0 "JP5" H 6250 2850 60  0000 C CNN
 F 1 "4_PIN_1" V 6350 2550 60  0000 C CNN
-F 2 "Pin_Headers:Pin_Header_Straight_1x04" H 6250 2550 60  0001 C CNN
+F 2 "tapmatrix:Pin_Header_Straight_1x04" H 6250 2550 60  0001 C CNN
 F 3 "" H 6250 2550 60  0000 C CNN
 	1    6250 2550
