File: kicad/tapMatrix_Shield/tapMatrix.sch (KiCad schematic (older format))
At the start: 29 parts, among them P5 TS_ZIF, P6 LED_MATRIX_HDR, U1 MCP1700T-3302E/MB, U2 MCP4921-E/SN, U3 74LS125, U4 TL072, U5 SD_CARD, U6 DS1307

Commit message: corrected JP4, where MATRIX_WR and MATRIX_DATA were reveresed
Changed lines of the file:
@@
 Sheet 1 1
 Title "tapMatrix Shield"
-Date "26 Oct 2014"
+Date "23 Nov 2014"
 Rev "0.3"
 Comp "Responsive Devices, Inc."
@@
 $EndComp
 Text Label 3600 2300 0    60   ~ 0
-MATRIX_DATA
+MATRIX_WR
 Text Label 8350 2000 0    60   ~ 0
 MATRIX_DATA
 Text Label 3600 2200 0    60   ~ 0
-MATRIX_WR
+MATRIX_DATA
 Text Label 8350 1850 0    60   ~ 0
 MATRIX_WR

Commit message: Schematic: replaced RTC and added pot replaced DS1207 with DS3231 real time clock added potentiometer to amplifier circuit
Parts:
- removed U6: DS1307, tapmatrix:SOIC-8_N, symbol DS1307
- added RV?: POT, symbol POT
- added U?: DS3231, symbol DS3231
- U4: value TL072 -> TS922
Connections:
- wire segments 137 -> 134
Other:
- note added: "Op Amp"
- note added: "Volume"
- note removed: "(VOLUME REMOVED)"
- note removed: "AMP"

Commit message: Updated schematic annotations
Parts:
- gave numbers to parts that had none: 2
