File: kicad/tapMatrix_Board/tapMatrix.sch (KiCad schematic (older format))
At the start: 35 parts, among them P5 TS_ZIF, P6 LED_MATRIX_HDR, U1 MCP1703, U2 MCP4921-E/SN, U3 74AHC125, U4 TS922, U5 SD_CARD, U6 DS3231

Commit message: complete first draft of 0.5 board
add headers for FTDI, I2C, other extra pins.
Parts:
- removed C? (x2): 47uF, tapmatrix:EEE-0JA101WR, symbol C
- removed JP7: 6_PIN_3, tapmatrix:Pin_Header_Straight_1x06, symbol 6_PIN_3
- added C10, C11: 47uF, symbol CP2
- added C13: 0.1uF, tapmatrix:C_0603, symbol C
- added D2: LED, symbol LED
- added JP1: FTDI, symbol 6_PIN_1
- added JP2: EXTRA, symbol 8_PIN_1
- added R6: 1.5K, tapmatrix:R_0603, symbol R
- added SW1: SW_PUSH, symbol SW_PUSH
- P1: renamed from P?; value BARREL_JACK -> +9V Power
- gave numbers to parts that had none: 5
Connections:
- net labels added: D8, D9, RESET
- wire segments 161 -> 181
- no-connect marks 13 -> 15
Other:
- note added: "5V Power Supply"
- note added: "Touchscreen ZIF Socket + Header"
- note added: "to do:\nconsider adding ICSP\nconsider adding some more LED’s for TX/RX, pin 13 (PB5, “SCK”)"
- note removed: "Touchscreen ZIF Socket + Optional Headers"

Commit message: Add ICSP header and power LED
Parts:
- added D3: LED, symbol LED
- added JP3: ICSP, symbol ICSP
- added R7: 510, tapmatrix:R_0603, symbol R
- R6: value 1.5K -> 510
Connections:
- wire segments 181 -> 193
Other:
- note added: "FTDI-USB goes here"
- note added: "to do:\nadd FTDI+USB option, including RX/TX LED’s\nverify LED’s-Resistors"
- note removed: "to do:\nconsider adding ICSP\nconsider adding some more LED’s for TX/RX, pin 13 (PB5, “SCK”)"
