File: kicad/tapMatrix_Board/tapMatrix.sch (KiCad schematic (older format))
At the start: 63 parts, among them P1 +9V Power, P5 TS_ZIF, P6 LED_MATRIX_HDR, SW1 SW_PUSH, U1 MCP1703, U2 MCP4921-E/SN, U3 74AHC125, U4 TS922, U5 SD_CARD, U6 DS3231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

Commit message: Add SPI header for nRF8001
Parts:
- removed JP2: EXTRA, symbol 8_PIN_1
- added JP2: nRF8001, symbol nRF8001
- added JP4: 4_PIN_2, symbol 4_PIN_2
- D4: renamed from D?; value RXLED -> TXLED
- gave numbers to parts that had none: 19
Connections:
- wire segments 251 -> 254
- no-connect marks 16 -> 26
Other:
- note added: "FTDI Header"
- note added: "I2C Header"
- note added: "ISCP Header"
- note added: "Real Time Clock"
- note added: "nRF8001 Header"
- note added: "to do:\nadd FTDI+USB option, including RX/TX LED’s (done!)\nverify LED’s-Resistors (to do: 1K? 510R?)\nadd header for nRF8001 (done 3/30/15)\nif nRF8001, swap back to DS1302? (do this after confirming nRF8001)"
- note removed: "REAL TIME CLOCK"
- note removed: "to do:\nadd FTDI+USB option, including RX/TX LED’s (done!)\nverify LED’s-Resistors (to do: 1K? 510R?)\nadd header for nRF8001?\nif nRF8001, swap back to DS1302?"

Commit message: Datasheets + Footprints for 5V supply circuit
Parts:
- C10, C11: footprint (none) -> tapmatrix:CAP_MVA_F55
- D1: footprint (none) -> tapmatrix:DS16004
- D2, D3: footprint (none) -> tapmatrix:D_0603
- P1: footprint (none) -> tapmatrix:PJ-102AH
- U7: footprint (none) -> tapmatrix:SOT223_318H
Changed lines of the file:
@@
 F 0 "P1" H 1150 1750 60  0000 C CNN
 F 1 "+9V Power" H 1150 1300 60  0000 C CNN
-F 2 "" H 1150 1500 60  0000 C CNN
+F 2 "tapmatrix:PJ-102AH" H 1150 1500 60  0001 C CNN
 F 3 "" H 1150 1500 60  0000 C CNN
 	1    1150 1500
@@
 F 0 "D1" H 2000 1500 40  0000 C CNN
 F 1 "DIODE" H 2000 1300 40  0000 C CNN
-F 2 "" H 2000 1400 60  0000 C CNN
+F 2 "tapmatrix:DS16004" H 2000 1400 60  0001 C CNN
 F 3 "" H 2000 1400 60  0000 C CNN
 	1    2000 1400
@@
 P 2950 1450
 F 0 "U7" H 2950 1700 40  0000 C CNN
-F 1 "NCP1117ST50T3G" H 2950 1650 40  0000 C CNN
-F 2 "" H 2950 1450 60  0000 C CNN
+F 1 "NCP1117ST50T3G" H 2950 1650 40  0001 C CNN
+F 2 "tapmatrix:SOT223_318H" H 2950 1450 60  0001 C CNN
 F 3 "" H 2950 1450 60  0000 C CNN
 	1    2950 1450
@@
 F 0 "D2" H 4600 1700 50  0000 C CNN
 F 1 "LED" H 4600 1500 50  0000 C CNN
-F 2 "" H 4600 1600 60  0000 C CNN
+F 2 "tapmatrix:D_0603" H 4600 1600 60  0001 C CNN
 F 3 "" H 4600 1600 60  0000 C CNN
 	1    4600 1600
@@
 F 0 "C10" H 2350 1700 40  0000 L CNN
 F 1 "47uF" H 2356 1515 40  0000 L CNN
-F 2 "" H 2388 1450 30  0000 C CNN
+F 2 "tapmatrix:CAP_MVA_F55" H 2388 1450 30  0001 C CNN
 F 3 "" H 2350 1600 60  0000 C CNN
 	1    2350 1600
@@
 F 0 "C11" H 3600 1700 40  0000 L CNN
 F 1 "47uF" H 3606 1515 40  0000 L CNN
-F 2 "" H 3638 1450 30  0000 C CNN
+F 2 "tapmatrix:CAP_MVA_F55" H 3638 1450 30  0001 C CNN
 F 3 "" H 3600 1600 60  0000 C CNN
 	1    3600 1600
@@
 F 0 "D3" H 5100 1700 50  0000 C CNN
 F 1 "LED" H 5100 1500 50  0000 C CNN
-F 2 "" H 5100 1600 60  0000 C CNN
+F 2 "tapmatrix:D_0603" H 5100 1600 60  0001 C CNN
 F 3 "" H 5100 1600 60  0000 C CNN
 	1    5100 1600

Commit message: Datasheets + Footprints for AT328p, XTAL, Fuse, USB, FTDI
Parts:
- C17: value 10uF -> 4.7uF; footprint (none) -> tapmatrix:EEE-0JA101WR
- F1: footprint (none) -> tapmatrix:Fuse_MF_MSMF
- P2: footprint (none) -> tapmatrix:USBMiniB_UX60_MB_5S8
- SW1: footprint (none) -> tapmatrix:SW_3BU_1000P
- U8: footprint TQFP32 -> Housings_QFP:TQFP-32_7x7mm_Pitch0.8mm
- U9: footprint (none) -> tapmatrix:SSOP20_FTDI231X
- X1: footprint (none) -> tapmatrix:XTAL_CSTCE_V
Connections:
- no-connect marks 26 -> 25

Commit message: cosmetic updates to schematic
Connections:
- wire segments 254 -> 257
Changed lines of the file:
@@
 	1    0    0    -1
 $EndComp
-$Comp
-L LED_MATRIX_HDR P6
-U 1 1 53F2DDF1
-P 10500 7850
-F 0 "P6" H 10500 8600 60  0000 C CNN
-F 1 "LED_MATRIX_HDR" H 10500 7150 50  0001 C CNN
-F 2 "tapmatrix:5103310­-3" H 10500 7850 60  0001 C CNN
-F 3 "http://www.te.com/commerce/DocumentDelivery/DDEController?Action=srchrtrv&DocNm=5103310&DocType=Customer+Drawing&DocLang=English" H 10500 7850 60  0001 C CNN
-	1    10500 7850
-	1    0    0    -1
-$EndComp
-NoConn ~ 9850 7450
-NoConn ~ 9850 7600
-NoConn ~ 9850 7900
 NoConn ~ 11100 7900
-NoConn ~ 11100 7450
-$Comp
-L GND #PWR43
-U 1 1 53F2DE59
-P 9600 7900
-F 0 "#PWR43" H 9600 7900 30  0001 C CNN
-F 1 "GND" H 9600 7830 30  0001 C CNN
-F 2 "" H 9600 7900 60  0000 C CNN
-F 3 "" H 9600 7900 60  0000 C CNN
-	1    9600 7900
-	1    0    0    -1
-$EndComp
-$Comp
-L GND #PWR55
-U 1 1 53F2E04E
-P 11500 8350
-F 0 "#PWR55" H 11500 8350 30  0001 C CNN
-F 1 "GND" H 11500 8280 30  0001 C CNN
-F 2 "" H 11500 8350 60  0000 C CNN
-F 3 "" H 11500 8350 60  0000 C CNN
-	1    11500 8350
-	1    0    0    -1
-$EndComp
 Text Notes 7450 10200 2    60   ~ 0
 Touchscreen ZIF Socket + Header
-Text Notes 10900 8650 2    60   ~ 0
+Text Notes 10900 8500 2    60   ~ 0
 LED Matrix Header
 $Comp
@@
 U 1 1 53F2E748
 P 14950 2400
-F 0 "U5" H 15000 3100 60  0000 C CNN
-F 1 "SD_CARD" H 14950 1700 60  0000 C CNN
+F 0 "U5" H 14950 2800 60  0000 C CNN
+F 1 "SD_CARD" H 14950 1950 60  0000 C CNN
 F 2 "tapmatrix:114-00841-68" H 14950 2600 60  0001 C CNN
 F 3 "" H 14950 2600 60  0000 C CNN
@@
 Text Notes 15350 3600 2    60   ~ 0
 MicroSD Card Socket
-NoConn ~ 14250 1900
-$Comp
-L GND #PWR70
-U 1 1 53F3050A
-P 16100 3000
-F 0 "#PWR70" H 16100 3000 30  0001 C CNN
-F 1 "GND" H 16100 2930 30  0001 C CNN
-F 2 "" H 16100 3000 60  0000 C CNN
-F 3 "" H 16100 3000 60  0000 C CNN
-	1    16100 3000
-	1    0    0    -1
-$EndComp
-NoConn ~ 15650 2500
 $Comp
 L GND #PWR65
 U 1 1 53F30748
-P 14100 3000
-F 0 "#PWR65" H 14100 3000 30  0001 C CNN
-F 1 "GND" H 14100 2930 30  0001 C CNN
-F 2 "" H 14100 3000 60  0000 C CNN
-F 3 "" H 14100 3000 60  0000 C CNN
-	1    14100 3000
+P 14100 2800
+F 0 "#PWR65" H 14100 2800 30  0001 C CNN
+F 1 "GND" H 14100 2730 30  0001 C CNN
+F 2 "" H 14100 2800 60  0000 C CNN
+F 3 "" H 14100 2800 60  0000 C CNN
+	1    14100 2800
 	1    0    0    -1
 $EndComp
@@
 	1    0    0    -1
 $EndComp
-Text Label 11200 7750 0    60   ~ 0
-MATRIX_DATA
-Text Label 11200 7600 0    60   ~ 0
-MATRIX_WR
-Text Label 11200 7300 0    60   ~ 0
-MATRIX_CS
-Text Label 9250 7300 0    60   ~ 0
-MATRIX_CLK
 $Comp
 L +5V #PWR44
 U 1 1 53F45B08
-P 9600 8200
-F 0 "#PWR44" H 9600 8290 20  0001 C CNN
-F 1 "+5V" H 9600 8290 30  0000 C CNN
-F 2 "" H 9600 8200 60  0000 C CNN
-F 3 "" H 9600 8200 60  0000 C CNN
-	1    9600 8200
+P 9500 8100
+F 0 "#PWR44" H 9500 8190 20  0001 C CNN
+F 1 "+5V" H 9500 8190 30  0000 C CNN
+F 2 "" H 9500 8100 60  0000 C CNN
+F 3 "" H 9500 8100 60  0000 C CNN
+	1    9500 8100
 	1    0    0    -1
 $EndComp
@@
 Text Label 5550 9950 0    60   ~ 0
 YM
-Text Label 15650 2300 0    60   ~ 0
-MISO
-Text Label 15650 1900 0    60   ~ 0
-SCLK
 Text Label 11300 2050 0    60   ~ 0
 SCLK
@@
 Text Label 13050 2050 0    60   ~ 0
 CS
-Text Label 13900 2100 0    60   ~ 0
-CS
-Text Label 13900 2300 0    60   ~ 0
-DATA_IN
 Text Label 11800 2050 0    60   ~ 0
 SD_CS
@@
 L +3.3V #PWR64
 U 1 1 53F5A65D
-P 13950 2500
-F 0 "#PWR64" H 13950 2460 30  0001 C CNN
-F 1 "+3.3V" H 13950 2610 30  0000 C CNN
-F 2 "" H 13950 2500 60  0000 C CNN
-F 3 "" H 13950 2500 60  0000 C CNN
-	1    13950 2500
+P 13800 2450
+F 0 "#PWR64" H 13800 2410 30  0001 C CNN
+F 1 "+3.3V" H 13800 2560 30  0000 C CNN
+F 2 "" H 13800 2450 60  0000 C CNN
+F 3 "" H 13800 2450 60  0000 C CNN
+	1    13800 2450
 	1    0    0    -1
 $EndComp
@@
 Wire Wire Line
 	-765750 -630000 -766100 -630000
-Wire Wire Line
-	9850 7750 9600 7750
-Wire Wire Line
-	9600 7750 9600 7900
-Wire Wire Line
-	9850 8050 9850 8350
-Connection ~ 9850 8200
-Wire Wire Line
-	11100 8050 11100 8350
-Connection ~ 11100 8200
-Wire Wire Line
-	11100 8200 11500 8200
-Wire Wire Line
-	11500 8200 11500 8350
-Wire Wire Line
-	15650 2100 16100 2100
-Wire Wire Line
-	16100 2100 16100 3000
-Wire Wire Line
-	15650 2700 16100 2700
-Connection ~ 16100 2700
-Wire Wire Line
-	15650 2900 16100 2900
-Connection ~ 16100 2900
-Wire Wire Line
-	14250 2700 14100 2700
-Wire Wire Line
-	14100 2700 14100 3000
-Wire Wire Line
-	14250 2900 14100 2900
-Connection ~ 14100 2900
 Connection ~ 12100 2050
 Wire Wire Line
-	11100 7750 11600 7750
-Wire Wire Line
-	11100 7600 11600 7600
-Wire Wire Line
-	11100 7300 11600 7300
-Wire Wire Line
-	9850 8200 9600 8200
-Wire Wire Line
 	11200 3000 11550 3000
 Wire Wire Line
@@
 	5800 9850 5550 9850
 Wire Wire Line
-	14250 2300 13900 2300
-Wire Wire Line
-	15650 2300 15950 2300
-Wire Wire Line
-	15650 1900 15950 1900
-Wire Wire Line
 	11200 2050 11550 2050
 Wire Wire Line
@@
 	13000 2050 13300 2050
 Wire Wire Line
-	14250 2100 13900 2100
-Wire Wire Line
 	12100 2050 11800 2050
-Wire Wire Line
-	13950 2500 14250 2500
 Wire Wire Line
 	9750 5400 9300 5400
@@
 Connection ~ 2450 3250
 Connection ~ 15500 5700
-Connection ~ 9850 7300
 Connection ~ 14000 5700
-Wire Wire Line
-	9250 7300 9850 7300
 Wire Wire Line
 	1100 3000 1100 3250
@@
 Text Notes 7450 8800 2    60   ~ 0
 FTDI Header
-Text Notes 13300 8650 2    60   ~ 0
+Text Notes 13300 8500 2    60   ~ 0
 ISCP Header
 $Comp
@@
 Text Label 14700 7950 0    60   ~ 0
 I2C_SCL
-Text Notes 15550 8650 2    60   ~ 0
+Text Notes 15500 8500 2    60   ~ 0
 I2C Header
 NoConn ~ 6350 5600
@@
 Wire Wire Line
 	5500 2100 5700 2100
+Wire Wire Line
+	14250 2650 14100 2650
+Wire Wire Line
+	14100 2550 14100 2800
+Wire Wire Line
+	14250 2550 14100 2550
+Connection ~ 14100 2650
+Wire Wire Line
+	14250 2450 13800 2450
+Wire Wire Line
+	14250 2350 13900 2350
+Text Label 13900 2350 0    60   ~ 0
+DATA_IN
+Wire Wire Line
+	14250 2250 13900 2250
+Text Label 13900 2250 0    60   ~ 0
+CS
+NoConn ~ 14250 2150
+$Comp
+L GND #PWR?
+U 1 1 551CEDD4
+P 16150 2800
+F 0 "#PWR?" H 16150 2800 30  0001 C CNN
+F 1 "GND" H 16150 2730 30  0001 C CNN
+F 2 "" H 16150 2800 60  0000 C CNN
+F 3 "" H 16150 2800 60  0000 C CNN
+	1    16150 2800
+	1    0    0    -1
+$EndComp
+Wire Wire Line
+	15650 2550 16150 2550
+Wire Wire Line
+	16150 2250 16150 2800
+Wire Wire Line
+	15650 2650 16150 2650
+Connection ~ 16150 2650
+Wire Wire Line
+	15650 2250 16150 2250
+Connection ~ 16150 2550
+NoConn ~ 15650 2450
+Wire Wire Line
+	15650 2350 15950 2350
+Text Label 15750 2350 0    60   ~ 0
+MISO
+Wire Wire Line
+	15650 2150 15950 2150
+Text Label 15700 2150 0    60   ~ 0
+SCLK
+Wire Wire Line
+	9850 8100 9500 8100
+Wire Wire Line
+	9850 8000 9700 8000
+Wire Wire Line
+	9700 8000 9700 8200
+Connection ~ 9700 8100
+Wire Wire Line
+	9700 8200 9850 8200
+NoConn ~ 9850 7900
+Wire Wire Line
+	9850 7500 9300 7500
+Text Label 9300 7500 0    60   ~ 0
+MATRIX_CLK
+NoConn ~ 9850 7600
+NoConn ~ 9850 7700
+$Comp
+L GND #PWR?
+U 1 1 551D1E10
+P 9300 8350
+F 0 "#PWR?" H 9300 8350 30  0001 C CNN
+F 1 "GND" H 9300 8280 30  0001 C CNN
+F 2 "" H 9300 8350 60  0000 C CNN
+F 3 "" H 9300 8350 60  0000 C CNN
+	1    9300 8350
+	1    0    0    -1
+$EndComp
+Wire Wire Line
+	9850 7800 9300 7800
+Wire Wire Line
+	9300 7800 9300 8350
+$Comp
+L LED_MATRIX_HDR P6
+U 1 1 53F2DDF1
+P 10500 7850
+F 0 "P6" H 10500 8400 60  0000 C CNN
+F 1 "LED_MATRIX_HDR" H 10500 7150 50  0001 C CNN
+F 2 "tapmatrix:5103310­-3" H 10500 7850 60  0001 C CNN
+F 3 "http://www.te.com/commerce/DocumentDelivery/DDEController?Action=srchrtrv&DocNm=5103310&DocType=Customer+Drawing&DocLang=English" H 10500 7850 60  0001 C CNN
+	1    10500 7850
+	1    0    0    -1
+$EndComp
+$Comp
+L GND #PWR?
+U 1 1 551D2A7F
+P 11300 8350
+F 0 "#PWR?" H 11300 8350 30  0001 C CNN
+F 1 "GND" H 11300 8280 30  0001 C CNN
+F 2 "" H 11300 8350 60  0000 C CNN
+F 3 "" H 11300 8350 60  0000 C CNN
+	1    11300 8350
+	1    0    0    -1
+$EndComp
+Wire Wire Line
+	11100 8100 11300 8100
+Wire Wire Line
+	11300 8000 11300 8350
+Wire Wire Line
+	11100 8200 11300 8200
+Connection ~ 11300 8200
+Wire Wire Line
+	11100 8000 11300 8000
+Connection ~ 11300 8100
+NoConn ~ 11100 7600
+Wire Wire Line
+	11100 7500 11700 7500
+Wire Wire Line
+	11100 7700 11700 7700
+Wire Wire Line
+	11100 7800 11700 7800
+Text Label 11200 7500 0    60   ~ 0
+MATRIX_CS
+Text Label 11200 7700 0    60   ~ 0
+MATRIX_WR
+Text Label 11200 7800 0    60   ~ 0
+MATRIX_DATA
 $EndSCHEMATC

Commit message: Complete footprint association and netlist definition
Parts:
- D4, D5: footprint (none) -> tapmatrix:D_0603
- JP1, JP2: footprint (none) -> tapmatrix:Pin_Header_Straight_1x06
- JP3, JP4: footprint (none) -> tapmatrix:Pin_Header_Straight_1x08
- U10: footprint SOT-323 -> tapmatrix:SOT-323
- U8: footprint Housings_QFP:TQFP-32_7x7mm_Pitch0.8mm -> tapmatrix:TQFP-32_7x7mm_Pitch0.8mm

Commit message: Modify JP2 from 6pin to 10pin header
Parts:
- JP2: footprint tapmatrix:Pin_Header_Straight_1x06 -> tapmatrix:Pin_Header_Straight_1x10
Changed lines of the file:
@@
 F 0 "JP2" H 10500 9750 60  0000 C CNN
 F 1 "nRF8001" H 10450 8550 60  0001 C CNN
-F 2 "tapmatrix:Pin_Header_Straight_1x06" H 10500 9300 60  0001 C CNN
+F 2 "tapmatrix:Pin_Header_Straight_1x10" H 10500 9300 60  0001 C CNN
 F 3 "" H 10500 9300 60  0000 C CNN
 	1    10500 9300

Commit message: Rough placement of footprints
Parts:
- JP3: footprint tapmatrix:Pin_Header_Straight_1x08 -> tapmatrix:Pin_Header_Straight_2x03
Changed lines of the file:
@@
 F 0 "JP3" H 13000 8150 50  0000 C CNN
 F 1 "ICSP" H 13000 7750 50  0000 C CNN
-F 2 "tapmatrix:Pin_Header_Straight_1x08" H 13000 6750 60  0001 C CNN
+F 2 "tapmatrix:Pin_Header_Straight_2x03" H 13000 6750 60  0001 C CNN
 F 3 "" H 13000 6750 60  0000 C CNN
 	1    13000 7950

Commit message: add C20, begin routing
Parts:
- added C20: 0.1uF, tapmatrix:C_0603, symbol C
Connections:
- wire segments 257 -> 260
Changed lines of the file:
@@
 Wire Wire Line
 	8100 5800 8550 5800
-Text Label 8250 5800 0    60   ~ 0
-RESET
 Wire Wire Line
 	6350 5800 7000 5800
@@
 Text Label 11200 7800 0    60   ~ 0
 MATRIX_DATA
+$Comp
+L C C20
+U 1 1 551FB47B
+P 8550 5250
+F 0 "C20" H 8550 5350 40  0000 L CNN
+F 1 "0.1uF" H 8556 5165 40  0000 L CNN
+F 2 "tapmatrix:C_0603" H 8588 5100 30  0001 C CNN
+F 3 "" H 8550 5250 60  0000 C CNN
+	1    8550 5250
+	1    0    0    -1
+$EndComp
+Wire Wire Line
+	8550 5800 8550 5450
+Wire Wire Line
+	8550 5050 8550 4500
+Wire Wire Line
+	8550 4500 9100 4500
+Text Label 8800 4500 0    60   ~ 0
+RESET
 $EndSCHEMATC
