File: kicad/tapMatrix_Board/tapMatrix.sch (KiCad schematic (older format))
At the start: 65 parts, among them P1 +9V Power, P2 USB-MINI-B, P5 TS_ZIF, P6 LED_MATRIX_HDR, SW1 SW_PUSH, U1 MCP1703, U10 2N7002PW, U2 MCP4921-E/SN, U3 74AHC125, U4 TS922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

Commit message: Complete first pass routing
Parts:
- JP4: footprint tapmatrix:Pin_Header_Straight_1x08 -> tapmatrix:Pin_Header_Straight_1x04
Changed lines of the file:
@@
 F 0 "JP4" H 15550 8400 60  0000 C CNN
 F 1 "4_PIN_2" H 15550 7600 60  0001 C CNN
-F 2 "tapmatrix:Pin_Header_Straight_1x08" H 15550 8000 60  0001 C CNN
+F 2 "tapmatrix:Pin_Header_Straight_1x04" H 15550 8000 60  0001 C CNN
 F 3 "" H 15550 8000 60  0000 C CNN
 	1    15550 8000

Commit message: Complete routing and formatting, create Gerbers
Changed lines of the file:
@@
 Sheet 1 1
 Title "tapMatrix Board"
-Date "1 Apr 2015"
+Date "9 Apr 2015"
 Rev "0.5"
 Comp "Responsive Devices, Inc."
